Commit message: bugfix to make it work

File: gazebo/gazebo.urdf.xacro (robot description, xacro)
@@ -2,5 +2,5 @@
 <robot xmlns:xacro="http://ros.org/wiki/xacro">
 <xacro:arg name="task_period" default="0.004" />
-<xacro:arg name="robot_name" default="starbot" />
+<xacro:arg name="robot_name" default="myrobot" />
 	<gazebo>
 		<plugin name="gazebo_ros_controller_manager" filename="libgazebo_ros_control.so">

File: robots/myrobot.urdf.xacro (robot description, xacro)
@@ -1,12 +1,12 @@
 <?xml version="1.0" ?>
-<robot name="starbot" xmlns:xacro="http://ros.org/wiki/xacro">
+<robot name="myrobot" xmlns:xacro="http://ros.org/wiki/xacro">
     <!--- new_gazebo_version should be false by default because pinocchio needs it!-->
-    <xacro:arg name="robot_name" default="starbot"/>
+    <xacro:arg name="robot_name" default="myrobot"/>
     <xacro:arg name="new_gazebo_version" default="false"/>
-    <xacro:include filename="$(find starbot_description)/gazebo/gazebo.urdf.xacro">
+    <xacro:include filename="$(find myrobot_description)/gazebo/gazebo.urdf.xacro">
         <xacro:arg name="task_period" value="$(arg task_period)"/>
 	<xacro:arg name="robot_name" value="$(arg robot_name)"/>
     </xacro:include>
-    <xacro:include filename="$(find starbot_description)/urdfs/leg.xacro"/>
+    <xacro:include filename="$(find myrobot_description)/urdfs/myleg.xacro"/>
     <!-- BASE LINK -->
     <!-- floating type is supported in older versions of Gazebo. In new Gazebo if a link has no parent, it is supposed to be attached to a floating joint -->

File: urdfs/myleg.gazebo.xacro (robot description, xacro)
@@ -14,5 +14,5 @@
                                 <update_rate>1000.0</update_rate>
                                 <contact>
-                                        <collision>${name}_XXXX</collision>
+                                        <collision>${name}_shoulder_link_collision</collision>
                                 </contact>
                                 <plugin name="${name}_foot_bumper" filename="libgazebo_ros_bumper.so">

File: urdfs/myleg.xacro (robot description, xacro)
@@ -6,28 +6,28 @@
     <!-- This macro has for purpose to define a leg -->
     <xacro:macro name="leg" params="name parent robot_name *origin ">
-	<joint name="${name}_shoulder_pan" type="revolute">
+	<joint name="${name}_shoulder_pan_joint" type="revolute">
 		<parent link="${parent}"/>
-		<child link="${name}_shoulder"/>
+		<child link="${name}_shoulder_link"/>
 		<axis xyz="0 0 1"/>
 		<xacro:insert_block name="origin"/>
 		<limit effort="50" velocity="10.0" lower="-3.14" upper="3.14" />
 	</joint>
-	<link name="${name}_shoulder">
+	<link name="${name}_shoulder_link">
 		<inertial>
-		<origin xyz="0.0 0.0 0.0"/>
+			<origin xyz="0.0 0.0 0.0"/>
 			<mass value="0.05" />
 			<inertia  ixx="0.001" ixy="0.0"  ixz="0.0"  iyy="0.001"  iyz="0.0"  izz="0.001" />
 		</inertial>
-		<visual>
-		<origin xyz="0 0.0 0.0" rpy="0 0 0"/>
-		<geometry>
-			<box size="0.1 0.1 0.2"/>
-		</geometry>
-		</visual>
+			<visual>
+			<origin xyz="0 0.0 0.0" rpy="0 0 0"/>
+			<geometry>
+				<box size="0.1 0.1 0.2"/>
+			</geometry>
+			</visual>
 		<collision>
-		<origin  xyz="0 0.0 0.0 " rpy="0 0 0"/>
-		<geometry>
-			<box size="0.1 0.1 0.2"/>
-		</geometry>
+			<origin  xyz="0 0.0 0.0 " rpy="0 0 0"/>
+			<geometry>
+				<box size="0.1 0.1 0.2"/>
+			</geometry>
 		</collision>
 	</link>

Commit message: removed trunk link to simplify

File: gazebo/gazebo.urdf.xacro (robot description, xacro)
@@ -12,5 +12,5 @@
 		<plugin filename="libgazebo_ros_p3d.so" name="gazebo_ros_p3d">
                         <robotNamespace>/$(arg robot_name)</robotNamespace>
-                        <bodyName>trunk</bodyName>
+                        <bodyName>base_link</bodyName>
 			<topicName>ground_truth</topicName>
 			<frameName>world</frameName>

File: robots/myrobot.urdf.xacro (robot description, xacro)
@@ -9,23 +9,6 @@
     </xacro:include>
     <xacro:include filename="$(find myrobot_description)/urdfs/myleg.xacro"/>
-    <!-- BASE LINK -->
-    <!-- floating type is supported in older versions of Gazebo. In new Gazebo if a link has no parent, it is supposed to be attached to a floating joint -->
-    <xacro:unless value="$(arg new_gazebo_version)">
-        <!-- Floating-base Joint -->
-        <link name="world"/>
-        <joint name="floating_base_joint" type="floating" >
-            <origin rpy="0 0 0" xyz="0 0 0"/>
-            <parent link="world"/>
-            <child link="base_link"/>
-        </joint>
-    </xacro:unless>
-    <link name="base_link" />
-    <joint name="floating_base" type="fixed">
-        <origin rpy="0 0 0" xyz="0 0 0"/>
-        <parent link="base_link"/>
-        <child link="trunk"/>
-    </joint>
-    <link name="trunk">
-	<inertial>
+    <link name="base_link">
+   	<inertial>
 		<origin xyz="0.0 0.0 0.0"/>
 		<mass value="15" />
